Commit message: Add a box as chassis

File: description/robot_core.xacro (robot description, xacro)
@@ -15,3 +15,17 @@
     <link name="base_link">
     </link>
+    <joint name="chassis_joint" type="fixed">
+        <parent link="base_link"/>
+        <child link="chassis"/>
+        <origin xyz="-0.1 0 0"/>
+    </joint>
+    <link name="chassis">
+        <visual>
+            <origin xyz="0.15 0 0.075" rpy="0 0 0"/>
+            <geometry>
+                <box size="0.3 0.3 0.15"/>
+            </geometry>
+            <material name="white"/>
+        </visual>
+    </link>
 </robot>

Commit message: Adding wheels

File: description/robot_core.xacro (robot description, xacro)
@@ -29,3 +29,47 @@
         </visual>
     </link>
+    <!-- LEFT WHEEL -->
+    <joint name="left_wheel_joint" type="continuous">
+        <parent link="base_link"/>
+        <child link="left_wheel"/>
+        <origin xyz="0 0.175 0" rpy="-${pi/2} 0 0"/>
+        <axis xyz="0 0 1"/>
+    </joint>
+    <link name="left_wheel">
+        <visual>
+            <geometry>
+                <cylinder length="0.04" radius="0.05" />/>
+            </geometry>
+            <material name="blue"/>
+        </visual>
+    </link>
+    <!-- RIGHT WHEEL -->
+    <joint name="right_wheel_joint" type="continuous">
+        <parent link="base_link"/>
+        <child link="right_wheel"/>
+        <origin xyz="0 -0.175 0" rpy="${pi/2} 0 0"/>
+        <axis xyz="0 0 -1"/>
+    </joint>
+    <link name="right_wheel">
+        <visual>
+            <geometry>
+                <cylinder length="0.04" radius="0.05" />/>
+            </geometry>
+            <material name="blue"/>
+        </visual>
+    </link>
+    <!-- CASTER WHEEL -->
+    <joint name="caster_wheel_joint" type="fixed">
+        <parent link="chassis"/>
+        <child link="caster_wheel"/>
+        <origin xyz="0.24 0 0" rpy="0 0 0"/>
+    </joint>
+    <link name="caster_wheel">
+        <visual>
+            <geometry>
+                <sphere radius="0.05" />
+            </geometry>
+            <material name="black"/>
+        </visual>
+    </link>
 </robot>

Commit message: Adding collision and using xacro properties

File: description/robot_core.xacro (robot description, xacro)
@@ -20,12 +20,22 @@
         <origin xyz="-0.1 0 0"/>
     </joint>
+    <xacro:property name="chassisOrigin" value="0.15 0 0.075" />
+    <xacro:property name="chassisGeometry" value="0.3 0.3 0.15" />
+    <xacro:property name="chassisMaterial" value="white" />
     <link name="chassis">
         <visual>
-            <origin xyz="0.15 0 0.075" rpy="0 0 0"/>
+            <origin xyz="${chassisOrigin}" rpy="0 0 0"/>
             <geometry>
-                <box size="0.3 0.3 0.15"/>
+                <box size="${chassisGeometry}"/>
             </geometry>
-            <material name="white"/>
+            <material name="${chassisMaterial}"/>
         </visual>
+        <collision>
+            <origin xyz="${chassisOrigin}" rpy="0 0 0"/>
+            <geometry>
+                <box size="${chassisGeometry}"/>
+            </geometry>
+            <material name="${chassisMaterial}"/>
+        </collision>
     </link>
     <!-- LEFT WHEEL -->
@@ -36,11 +46,20 @@
         <axis xyz="0 0 1"/>
     </joint>
+    <xacro:property name="leftWheelLength" value="0.04" />
+    <xacro:property name="leftWheelRadius" value="0.05" />
+    <xacro:property name="leftWheelMaterial" value="blue" />
     <link name="left_wheel">
         <visual>
             <geometry>
-                <cylinder length="0.04" radius="0.05" />/>
+                <cylinder length="${leftWheelLength}" radius="${leftWheelRadius}" />/>
             </geometry>
-            <material name="blue"/>
+            <material name="${leftWheelMaterial}"/>
         </visual>
+        <collision>
+            <geometry>
+                <cylinder length="${leftWheelLength}" radius="${leftWheelRadius}" />/>
+            </geometry>
+            <material name="${leftWheelMaterial}"/>
+        </collision>
     </link>
     <!-- RIGHT WHEEL -->
@@ -51,11 +70,20 @@
         <axis xyz="0 0 -1"/>
     </joint>
+    <xacro:property name="rightWheelLength" value="0.04" />
+    <xacro:property name="rightWheelRadius" value="0.05" />
+    <xacro:property name="rightWheelMaterial" value="blue" />
     <link name="right_wheel">
         <visual>
             <geometry>
-                <cylinder length="0.04" radius="0.05" />/>
+                <cylinder length="${rightWheelLength}" radius="${rightWheelRadius}" />/>
             </geometry>
-            <material name="blue"/>
+            <material name="${rightWheelMaterial}"/>
         </visual>
+        <collision>
+            <geometry>
+                <cylinder length="${rightWheelLength}" radius="${rightWheelRadius}" />/>
+            </geometry>
+            <material name="${rightWheelMaterial}"/>
+        </collision>
     </link>
     <!-- CASTER WHEEL -->
@@ -65,11 +93,19 @@
         <origin xyz="0.24 0 0" rpy="0 0 0"/>
     </joint>
+    <xacro:property name="casterWheelRadius" value="0.05" />
+    <xacro:property name="casterWheelMaterial" value="black" />
     <link name="caster_wheel">
         <visual>
             <geometry>
-                <sphere radius="0.05" />
+                <sphere radius="${casterWheelRadius}" />
             </geometry>
-            <material name="black"/>
+            <material name="${casterWheelMaterial}"/>
         </visual>
+        <collision>
+            <geometry>
+                <sphere radius="${casterWheelRadius}" />
+            </geometry>
+            <material name="${casterWheelMaterial}"/>
+        </collision>
     </link>
 </robot>

Commit message: Adding inertial for robot

File: description/robot_core.xacro (robot description, xacro)
@@ -1,4 +1,5 @@
 <?xml version="1.0"?>
 <robot xmlns:xacro="http://www.ros.org/wiki/xacro">
+    <xacro:include filename="inertial_macros.xacro" />
     <material name="white">
         <color rgba="1 1 1 1"/>
@@ -38,4 +39,7 @@
             <material name="${chassisMaterial}"/>
         </collision>
+        <xacro:inertial_box mass="0.5" x="0.3" y="0.3" z="0.15">
+            <origin xyz="0.15 0 0.075" rpy="0 0 0"/>
+        </xacro:inertial_box>
     </link>
     <!-- LEFT WHEEL -->
@@ -62,4 +66,7 @@
             <material name="${leftWheelMaterial}"/>
         </collision>
+        <xacro:inertial_cylinder mass="0.1" length="0.04" radius="0.05">
+            <origin xyz="0 0 0" rpy="0 0 0"/>
+        </xacro:inertial_cylinder>
     </link>
     <!-- RIGHT WHEEL -->
@@ -86,4 +93,7 @@
             <material name="${rightWheelMaterial}"/>
         </collision>
+        <xacro:inertial_cylinder mass="0.1" length="0.04" radius="0.05">
+            <origin xyz="0 0 0" rpy="0 0 0"/>
+        </xacro:inertial_cylinder>
     </link>
     <!-- CASTER WHEEL -->
@@ -108,4 +118,7 @@
             <material name="${casterWheelMaterial}"/>
         </collision>
+        <xacro:inertial_sphere mass="0.1" radius="0.05">
+            <origin xyz="0 0 0" rpy="0 0 0"/>
+        </xacro:inertial_sphere>
     </link>
 </robot>

Commit message: Changing robot's chassis to cylinder instead of box

File: description/robot_core.xacro (robot description, xacro)
@@ -19,8 +19,9 @@
         <parent link="base_link"/>
         <child link="chassis"/>
-        <origin xyz="-0.1 0 0"/>
+        <origin xyz="0 0 0"/>
     </joint>
-    <xacro:property name="chassisOrigin" value="0.15 0 0.075" />
-    <xacro:property name="chassisGeometry" value="0.3 0.3 0.15" />
+    <xacro:property name="chassisOrigin" value="0.04 0 0.04" />
+    <xacro:property name="chassisLength" value="0.08" />
+    <xacro:property name="chassisRadius" value="0.175" />
     <xacro:property name="chassisMaterial" value="white" />
     <link name="chassis">
@@ -28,5 +29,5 @@
             <origin xyz="${chassisOrigin}" rpy="0 0 0"/>
             <geometry>
-                <box size="${chassisGeometry}"/>
+                <cylinder length="${chassisLength}" radius="${chassisRadius}"/>
             </geometry>
             <material name="${chassisMaterial}"/>
@@ -35,10 +36,10 @@
             <origin xyz="${chassisOrigin}" rpy="0 0 0"/>
             <geometry>
-                <box size="${chassisGeometry}"/>
+                <cylinder length="${chassisLength}" radius="${chassisRadius}"/>
             </geometry>
             <material name="${chassisMaterial}"/>
         </collision>
         <xacro:inertial_box mass="0.5" x="0.3" y="0.3" z="0.15">
-            <origin xyz="0.15 0 0.075" rpy="0 0 0"/>
+            <origin xyz="${chassisOrigin}" rpy="0 0 0"/>
         </xacro:inertial_box>
     </link>
@@ -47,5 +48,5 @@
         <parent link="base_link"/>
         <child link="left_wheel"/>
-        <origin xyz="0 0.175 0" rpy="-${pi/2} 0 0"/>
+        <origin xyz="0 0.09 0" rpy="-${pi/2} 0 0"/>
         <axis xyz="0 0 1"/>
     </joint>
@@ -74,5 +75,5 @@
         <parent link="base_link"/>
         <child link="right_wheel"/>
-        <origin xyz="0 -0.175 0" rpy="${pi/2} 0 0"/>
+        <origin xyz="0 -0.09 0" rpy="${pi/2} 0 0"/>
         <axis xyz="0 0 -1"/>
     </joint>
@@ -101,5 +102,5 @@
         <parent link="chassis"/>
         <child link="caster_wheel"/>
-        <origin xyz="0.24 0 0" rpy="0 0 0"/>
+        <origin xyz="0.15 0 0" rpy="0 0 0"/>
     </joint>
     <xacro:property name="casterWheelRadius" value="0.05" />

Commit message: Adding launch file

File: description/robot_core.xacro (robot description, xacro)
@@ -44,4 +44,7 @@
         </xacro:inertial_cylinder>
     </link>
+    <gazebo reference="chassis">
+        <material>Gazebo/White</material>
+    </gazebo>
     <!-- LEFT WHEEL -->
     <joint name="left_wheel_joint" type="continuous">
@@ -71,4 +74,7 @@
         </xacro:inertial_cylinder>
     </link>
+    <gazebo reference="left_wheel">
+        <material>Gazebo/Blue</material>
+    </gazebo>
     <!-- RIGHT WHEEL -->
     <joint name="right_wheel_joint" type="continuous">
@@ -98,4 +104,7 @@
         </xacro:inertial_cylinder>
     </link>
+    <gazebo reference="right_wheel">
+        <material>Gazebo/Blue</material>
+    </gazebo>
     <!-- CASTER WHEEL -->
     <joint name="caster_wheel_joint" type="fixed">
@@ -123,3 +132,6 @@
         </xacro:inertial_sphere>
     </link>
+    <gazebo reference="caster_wheel">
+        <material>Gazebo/Black</material>
+    </gazebo>
 </robot>

Commit message: Adding simulated lidar sensor

File: description/robot_core.xacro (robot description, xacro)
@@ -14,4 +14,7 @@
         <color rgba="0 0 0 1"/>
     </material>
+    <material name="red">
+        <color rgba="1 0 0 1"/>
+<   /material>
     <link name="base_link">
     </link>
