Commit message: Fix an error

File: description/lidar.xacro (robot description, xacro)
@@ -24,5 +24,29 @@
     <gazebo reference="laser_frame">
         <material>Gazebo/Red</material>
-        ... About to put stuff here ...
+        <sensor name="laser" type="ray">
+            <pose> 0 0 0 0 0 0 </pose>
+            <visualize>true</visualize>
+            <update_rate>10</update_rate>
+            <ray>
+                <scan>
+                    <horizontal>
+                        <samples>360</samples>
+                        <min_angle>-3.14</min_angle>
+                        <max_angle>3.14</max_angle>
+                    </horizontal>
+                </scan>
+                <range>
+                    <min>0.3</min>
+                    <max>12</max>
+                </range>
+            </ray>
+            <plugin name="laser_controller" filename="libgazebo_ros_ray_sensor.so">
+                <ros>
+                    <argument>~/out:=scan</argument>
+                </ros>
+                <output_type>sensor_msgs/LaserScan</output_type>
+                <frame_name>laser_frame</frame_name>
+            </plugin>
+        </sensor>
     </gazebo>
 </robot>

File: description/robot_core.xacro (robot description, xacro)
@@ -16,5 +16,5 @@
     <material name="red">
         <color rgba="1 0 0 1"/>
-<   /material>
+    </material>
     <link name="base_link">
     </link>

Commit message: Functional mapping, saving and loading robot with lidar

File: description/lidar.xacro (robot description, xacro)
@@ -4,5 +4,5 @@
         <parent link="chassis"/>
         <child link="laser_frame"/>
-        <origin xyz="0.1 0 0.175" rpy="0 0 0"/>
+        <origin xyz="0.1 0 0.1" rpy="0 0 0"/>
     </joint>
     <link name="laser_frame">
@@ -37,5 +37,5 @@
                 </scan>
                 <range>
-                    <min>0.3</min>
+                    <min>0.1</min>
                     <max>12</max>
                 </range>

File: description/robot_core.xacro (robot description, xacro)
@@ -17,4 +17,12 @@
         <color rgba="1 0 0 1"/>
     </material>
+    <!-- BASE_FOOTPRINT LINK -->
+    <joint name="base_footprint_joint" type="fixed">
+        <parent link="base_link"/>
+        <child link="base_footprint"/>
+        <origin xyz="0 0 0" rpy="0 0 0"/>
+    </joint>
+    <link name="base_footprint">
+    </link>
     <link name="base_link">
     </link>
